Commit message: some examples but need fix on g1 init

File: data/robots/g1/g1_29dof_rev_1_0.urdf (robot description, URDF)
Before this commit: robot g1_29dof_rev_1_0, 39 links, 38 joints
Links:
- removed link pelvis
- added link base, mass 3.813; visual mesh filename=meshes/pelvis.STL
Joints:
- joint imu_in_pelvis_joint: parent pelvis -> base
- joint left_hip_pitch_joint: parent pelvis -> base
- joint pelvis_contour_joint: parent pelvis -> base
- joint right_hip_pitch_joint: parent pelvis -> base
- joint waist_yaw_joint: parent pelvis -> base
